Commit message: Fix camera orientation: was looking back at the arm, not the field
Debug frames showed the wrist camera staring at the robot's own forearm with
grey sky behind (meanBGR=(79,79,79), 0 weed pixels in every frame). gz cameras
look along their +X axis; rpy pitch +1.5708 mapped +X onto tool0 -Z (up/back at
the arm). Flipped to -1.5708 so +X aligns with tool0 +Z and the camera looks
DOWN at the field. Updated test_urdf accordingly.

Co-Authored-By: Claude Opus 4.8 <noreply@anthropic.com>

File: src/watermelon_demo/urdf/ur5_with_sensors.urdf.xacro (robot description, xacro)
@@ -37,8 +37,12 @@
     </inertial>
   </link>
+  <!-- rpy pitch of -1.5708 (negative 90 deg about Y). gz cameras look along
+       their +X axis, so this aligns the optical axis with tool0 +Z (the tool
+       approach axis) and the camera looks DOWN at the field. A pitch of
+       +1.5708 pointed it along tool0 -Z, back at the arm (wrong way). -->
   <joint name="tool0_to_camera" type="fixed">
     <parent link="tool0"/>
     <child link="camera_link"/>
-    <origin xyz="0.02 0.0 0.05" rpy="0 1.5708 0"/>
+    <origin xyz="0.02 0.0 0.05" rpy="0 -1.5708 0"/>
   </joint>
   <!-- Gazebo camera sensor attached to camera_link -->
